File: ZX80_Board.kicad_sch (KiCad schematic)
At the start: 124 parts, among them IC1 Z80, IC10 74LS365, IC11 74LS00, IC12 74LS00, IC13 74LS04, IC14 74LS05, IC15 74LS05, IC16 74LS10, IC17 74LS32, IC18 74LS74, IC19 74LS74, IC2 8332, IC20 74LS86, IC21 74LS93, IC22 7805C, IC3 2114, IC4 2114-1, IC5 74LS373, IC6 74LS157, IC7 74LS157, IC8 74LS157, IC9 74LS165, J1 9V-11V, J2 EAR, J3 MIC, SW1 1, SW10 0, SW11 Q, SW12 W, SW13 E, SW14 R, SW15 T, SW16 Y, SW17 U, SW18 I, SW19 O, SW2 2, SW20 P, SW21 A, SW22 S, SW23 D, SW24 F, SW25 G, SW26 H, SW27 J, SW28 K, SW29 L, SW3 3, SW30 NEW LINE, SW31 SHIFT, SW32 Z, SW33 X, SW34 C, SW35 V, SW36 B, SW37 N, SW38 M, SW39 •, SW4 4, SW40 SPACE, SW5 5, SW6 6, SW7 7, SW8 8, SW9 9, X1 6.5M

Commit message: Update 21/08/23
Parts:
- C1, C12, C13, C2, C4, C5, C6: footprint Capacitor_THT:C_Disc_D5.0mm_W2.5mm_P2.50mm -> Capacitor_THT:C_Disc_D6.0mm_W2.5mm_P5.00mm
- C11, C14, C9: footprint Capacitor_THT:C_Disc_D5.0mm_W2.5mm_P2.50mm -> Capacitor_THT:C_Disc_D3.4mm_W2.1mm_P2.50mm
- C15: footprint Capacitor_THT:C_Disc_D5.0mm_W2.5mm_P2.50mm -> Capacitor_THT:C_Disc_D3.0mm_W1.6mm_P2.50mm
- R1, R10, R11, R12, R13, R14, R15, R16, R17, R18, R19, R2, R20, R21, R22, R23, R24, R25, R27, R28, R29, R3, R30, R31, R32, R33, R34, R35, R4, R5, R6, R7, R8, R9: footprint Resistor_THT:R_Axial_DIN0207_L6.3mm_D2.5mm_P7.62mm_Horizontal -> ZX80:ZX80_R_Bare_Metal_Element_L12.4mm_W4.8mm_P11.40mm
Connections:
- net 0V: now also J1.T (TIP), J2.T (TIP), J3.T (TIP), RF_MODULATOR1.3 (0V); no longer J1.S (SLEEVE), J2.S (SLEEVE), J3.S (SLEEVE), RF_MODULATOR1.2 (0V)
- net 5V: now also EdgeConnector1.12A (~{NMI}), J2.S (SLEEVE), J3.S (SLEEVE); no longer C8.1, EdgeConnector1.2B (9V), IC22.1 (IN), J1.T (TIP), J2.T (TIP), J3.T (TIP), RF_MODULATOR1.1 (5V)
- net A0: no longer D4.2 (K), D5.2 (K), D6.2 (K), D7.2 (K), D8.2 (K), EdgeConnector1.10B (A3), EdgeConnector1.11A (~{INT}), EdgeConnector1.11B (A15), EdgeConnector1.12B (A14), EdgeConnector1.13B (A13), EdgeConnector1.14B (A12), EdgeConnector1.15B (A11), EdgeConnector1.16B (A10), EdgeConnector1.17B (A9), EdgeConnector1.18B (A8), EdgeConnector1.19B (A7), EdgeConnector1.20B (A6), EdgeConnector1.21B (A5), EdgeConnector1.22B (A4), EdgeConnector1.8B (A1), EdgeConnector1.9B (A2), IC1.1 (A11), IC1.16 (~{INT}), IC1.2 (A12), IC1.3 (A13), IC1.31 (A1), IC1.32 (A2), IC1.33 (A3), IC1.34 (A4), IC1.35 (A5), IC1.36 (A6), IC1.37 (A7), IC1.38 (A8), IC1.39 (A9), IC1.4 (A14), IC1.40 (A10), IC1.5 (A15), IC2.18 (A11), IC2.19 (A10), IC2.21 (CS2), IC2.22 (A9), IC3.1 (A6), IC3.15 (A9), IC3.16 (A8), IC3.17 (A7), IC3.2 (A5), IC3.3 (A4), IC3.4 (A3), IC3.5 (A2), IC3.6 (A1), IC4.1 (A6), IC4.15 (A9), IC4.16 (A8), IC4.17 (A7), IC4.2 (A5), IC4.3 (A4), IC4.4 (A3), IC4.5 (A2), IC4.6 (A1), IC6.10 (B), IC6.11 (A), IC6.13 (B), IC6.14 (A), IC6.3 (B), IC7.10 (B), IC7.13 (B), IC7.3 (B), IC7.6 (B), IC8.13 (B), IC8.3 (B), IC8.6 (B)
- net ~{A3}: now reaches IC2.5 (~{A3}), IC8.4 (A)
- net ~{A2}: now reaches IC2.6 (~{A2}), IC8.12 (B)
- net ~{A1}: now reaches IC2.7 (~{A1}), IC8.7 (A)
- net ~{A0}: now reaches IC2.8 (~{A0}), IC8.9 (B)
- net A14' renamed ~{A14}
- net A15' renamed ~{A15}
- net A8' renamed ~{A8}
- removed net D0': EdgeConnector1.10A (D4'), EdgeConnector1.1A (D7'), EdgeConnector1.4A (D0'), EdgeConnector1.5A (D1'), EdgeConnector1.6A (D2'), EdgeConnector1.7A (D6'), EdgeConnector1.8A (D5'), EdgeConnector1.9A (D3'), IC13.5, IC2.10 (D1'), IC2.11 (D2'), IC2.13 (D3'), IC2.14 (D4'), IC2.15 (D5'), IC2.16 (D6'), IC2.17 (D7'), IC2.9 (D0'), IC3.11 (D2'), IC3.12 (D0'), IC3.13 (D1'), IC3.14 (D7'), IC4.11 (D6'), IC4.12 (D5'), IC4.13 (D3'), IC4.14 (D4'), IC5.13 (D4), IC5.14 (D5), IC5.17 (D1), IC5.18 (D2), IC5.3 (D3), IC5.4 (D5), IC5.7 (D0), R10.1, R11.1, R28.1, R4.1, R5.1, R6.1, R7.1, R8.1, R9.1
- net ~{NMI}: no longer names the net of IC1.17 (~{NMI}), R12.2
- net ~{NMI}: no longer EdgeConnector1.12A (~{NMI})
- new net: R31.2, R32.1, RF_MODULATOR1.2 (~{SYNC})
- new net: R30.1, R33.1, RF_MODULATOR1.1 (VIDEO)
- new net 9V: C8.1, EdgeConnector1.2B (9V), IC22.1 (IN), J1.S (SLEEVE)
- new net A1: EdgeConnector1.8B (A1), IC1.31 (A1), IC3.6 (A1), IC4.6 (A1), IC8.6 (B)
- new net A10: D5.2 (K), EdgeConnector1.16B (A10), IC1.40 (A10), IC2.19 (A10)
- new net A11: D6.2 (K), EdgeConnector1.15B (A11), IC1.1 (A11), IC2.18 (A11)
- new net A12: D7.2 (K), EdgeConnector1.14B (A12), IC1.2 (A12), IC2.21 (CS2)
- new net A13: D8.2 (K), EdgeConnector1.13B (A13), IC1.3 (A13)
- new net A14: EdgeConnector1.12B (A14), IC1.4 (A14), IC6.10 (B), IC6.11 (A)
- new net A15: EdgeConnector1.11B (A15), IC1.5 (A15), IC6.13 (B), IC6.14 (A)
- new net A2: EdgeConnector1.9B (A2), IC1.32 (A2), IC3.5 (A2), IC4.5 (A2), IC8.13 (B)
- new net A3: EdgeConnector1.10B (A3), IC1.33 (A3), IC3.4 (A3), IC4.4 (A3), IC8.3 (B)
- new net A4: EdgeConnector1.22B (A4), IC1.34 (A4), IC3.3 (A4), IC4.3 (A4), IC7.10 (B)
- new net A5: EdgeConnector1.21B (A5), IC1.35 (A5), IC3.2 (A5), IC4.2 (A5), IC7.6 (B)
- new net A6: EdgeConnector1.11A (~{INT}), EdgeConnector1.20B (A6), IC1.16 (~{INT}), IC1.36 (A6), IC3.1 (A6), IC4.1 (A6), IC7.3 (B)
- new net A7: EdgeConnector1.19B (A7), IC1.37 (A7), IC3.17 (A7), IC4.17 (A7), IC7.13 (B)
- new net A8: EdgeConnector1.18B (A8), IC1.38 (A8), IC3.16 (A8), IC4.16 (A8), IC6.3 (B)
- new net A9: D4.2 (K), EdgeConnector1.17B (A9), IC1.39 (A9), IC2.22 (A9), IC3.15 (A9), IC4.15 (A9)
- new net ~{D0}: EdgeConnector1.4A (~{D0}), IC2.9 (~{D0}), IC3.12 (~{D0}), IC5.7 (D0), R10.1
- new net ~{D1}: EdgeConnector1.5A (~{D1}), IC2.10 (~{D1}), IC3.13 (~{D1}), IC5.14 (D5), R11.1
- new net ~{D2}: EdgeConnector1.6A (~{D2}), IC2.11 (~{D2}), IC3.11 (~{D2}), IC5.17 (D1), R8.1
- new net ~{D3}: EdgeConnector1.9A (~{D3}), IC2.13 (~{D3}), IC4.13 (~{D3}), IC5.18 (D2), R5.1
- new net ~{D4}: EdgeConnector1.10A (~{D4}), IC2.14 (~{D4}), IC4.14 (~{D4}), IC5.3 (D3), R4.1
- new net ~{D5}: EdgeConnector1.8A (~{D5}), IC2.15 (~{D5}), IC4.12 (~{D5}), IC5.4 (D5), R6.1
- new net ~{D6}: EdgeConnector1.7A (~{D6}), IC13.5, IC2.16 (~{D6}), IC4.11 (~{D6}), R28.1, R7.1
- new net ~{D7}: EdgeConnector1.1A (~{D7}), IC2.17 (~{D7}), IC3.14 (~{D7}), IC5.13 (D4), R9.1
Other:
- note added: "5V"
- note removed: "A0 - A15"
- note removed: "D0' - D7'"
